File: Board/BoardBoatV1.kicad_sch (KiCad schematic)
At the start: 16 parts, among them J1 GPIO, J2 Analog 1-3, J3 Motor1, J4 Motor2, J5 Switch1, J6 Switch2, J7 Switch3, U2 MCP3428

Commit message: gpio
Connections:
- net GPIO[18]/PCM.CLK is gone; now on net PWM2: J1.12 (Pin_12)
- net PWM2: no longer J1.32 (Pin_32)
Changed lines of the file:
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@@
-    (stroke (width 0) (type default) (color 0 0 0 0))
-  )
-  (wire (pts (xy 120.65 127) (xy 162.56 127))
     (stroke (width 0) (type default) (color 0 0 0 0))
   )
@@
     (stroke (width 0) (type solid) (color 0 0 0 0))
   )
+  (wire (pts (xy 120.65 127) (xy 147.32 127))
+    (stroke (width 0) (type default) (color 0 0 0 0))
+  )
   (wire (pts (xy 43.18 163.83) (xy 43.18 166.37))
     (stroke (width 0) (type default) (color 0 0 0 0))
@@
     (stroke (width 0) (type default) (color 0 0 0 0))
   )
-  (wire (pts (xy 120.65 101.6) (xy 147.32 101.6))
+  (wire (pts (xy 120.65 101.6) (xy 151.13 101.6))
     (stroke (width 0) (type solid) (color 0 0 0 0))
   )
@@
     )
   )
-  (global_label "PWM2" (shape input) (at 162.56 127 0) (fields_autoplaced)
+  (global_label "PWM2" (shape input) (at 151.13 101.6 0) (fields_autoplaced)
     (effects (font (size 1.27 1.27)) (justify left))
-    (property "Intersheet References" "${INTERSHEET_REFS}" (id 0) (at 170.546 127.0794 0)
+    (property "Intersheet References" "${INTERSHEET_REFS}" (id 0) (at 159.116 101.6794 0)
       (effects (font (size 1.27 1.27)) (justify left) hide)
     )
